File: PCB/RP2040-Guide.kicad_sch (KiCad schematic)
At the start: 35 parts, among them J1 USB_C_Receptacle_USB2.0, J2 SWD, J3 Conn_01x11, J4 Conn_01x11, J5 Conn_01x11, SW1 SW_Push, U1 W25Q128JVS, U2 USBLC6-2SC6, U3 RP2040, U4 XC6206PxxxMR-Regulator_Linear, Y1 12MHz

Commit message: Edit formatting on readme/pcb/schematic
Other:
- company: (none) -> Sleepdealer
- title: (none) -> RP2040 - Design Guide
Changed lines of the file:
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@@
 (kicad_sch (version 20210621) (generator eeschema)
   (paper "A4")
+  (title_block
+    (title "RP2040 - Design Guide")
+    (date "2021-12-07")
+    (rev "0.1")
+    (company "Sleepdealer")
+  )
   (junction (at 213.995 92.71) (diameter 0) (color 0 0 0 0))
   (junction (at 188.595 85.09) (diameter 0) (color 0 0 0 0))

Commit message: Update guide (Thanks xyz!)
Parts:
- added C7: 10uF, Capacitor_SMD:C_0402_1005Metric, symbol Device:C_Small
- R5, R6: footprint Resistor_SMD:R_0603_1608Metric -> Resistor_SMD:R_0402_1005Metric; LCSC C25190 -> C413051
- renumbered C9 to C10, C10 to C11, C11 to C12, C12 to C13, C13 to C14, C14 to C15, C15 to C16, C16 to C17, C7 to C8, C8 to C9, R2 to R1, R1 to R2
Connections:
- net +3V3: now also C7.1
- net GND: now also C7.2
Other:
- moved on the sheet: C10, C11, C12, C13, C14, C15, C8, C9

Commit message: Update BOM and borked vias (Thanks to SpeedyPotato!)
Parts:
- R5, R6: footprint Resistor_SMD:R_0402_1005Metric -> Resistor_SMD:R_0603_1608Metric; LCSC C413051 -> C25190
- Y1: LCSC C97242 -> C9002
Changed lines of the file:
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@@
       (effects (font (size 1.27 1.27)) hide)
     )
-    (property "LCSC" "C97242" (id 4) (at 192.405 60.96 0)
+    (property "LCSC" "C9002" (id 4) (at 192.405 60.96 0)
       (effects (font (size 1.27 1.27)) hide)
     )
@@
     (property "Reference" "R5" (id 0) (at 34.29 43.18 90))
     (property "Value" "27R" (id 1) (at 41.91 43.18 90))
-    (property "Footprint" "Resistor_SMD:R_0402_1005Metric" (id 2) (at 38.1 44.45 0)
+    (property "Footprint" "Resistor_SMD:R_0603_1608Metric" (id 2) (at 38.1 44.45 0)
       (effects (font (size 1.27 1.27)) hide)
     )
@@
       (effects (font (size 1.27 1.27)) hide)
     )
-    (property "LCSC" "C413051" (id 4) (at 38.1 44.45 0)
+    (property "LCSC" "C25190" (id 4) (at 38.1 44.45 0)
       (effects (font (size 1.27 1.27)) hide)
     )
@@
     (property "Reference" "R6" (id 0) (at 34.29 45.72 90))
     (property "Value" "27R" (id 1) (at 41.91 45.72 90))
-    (property "Footprint" "Resistor_SMD:R_0402_1005Metric" (id 2) (at 38.1 46.99 0)
+    (property "Footprint" "Resistor_SMD:R_0603_1608Metric" (id 2) (at 38.1 46.99 0)
       (effects (font (size 1.27 1.27)) hide)
     )
@@
       (effects (font (size 1.27 1.27)) hide)
     )
-    (property "LCSC" "C413051" (id 4) (at 38.1 46.99 0)
+    (property "LCSC" "C25190" (id 4) (at 38.1 46.99 0)
       (effects (font (size 1.27 1.27)) hide)
     )
@@
     )
     (path "/a17b7ec4-d21c-45d8-800e-1b60a1a1f0ec"
-      (reference "R5") (unit 1) (value "27R") (footprint "Resistor_SMD:R_0402_1005Metric")
+      (reference "R5") (unit 1) (value "27R") (footprint "Resistor_SMD:R_0603_1608Metric")
     )
     (path "/ab9374ae-9988-4ee9-bc8f-de5f61539e5f"
-      (reference "R6") (unit 1) (value "27R") (footprint "Resistor_SMD:R_0402_1005Metric")
+      (reference "R6") (unit 1) (value "27R") (footprint "Resistor_SMD:R_0603_1608Metric")
     )
     (path "/ecbc8a8f-d023-438f-b602-92f47848ee21"

Commit message: Update guide a bit
Parts:
- R2: value 10k -> (none); footprint Resistor_SMD:R_0402_1005Metric -> (none); LCSC C25744 -> C11702
Other:
- note removed: "You can probalby replace R1 with a 1k resistor to use simplify the BOM. Not sure why I didn't do that"
Changed lines of the file:
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@@
     (stroke (width 0) (type default) (color 0 0 0 0))
-  )
-  (text "You can probalby replace R1 with a 1k resistor\nto use simplify the BOM.\nNot sure why I didn't do that"
-    (at 16.51 20.32 0)
-    (effects (font (size 1.27 1.27)) (justify left bottom))
   )
   (text "MOUNTINGHOLES\n  (REMOVED)" (at 123.19 67.31 0)
@@
       (effects (font (size 1.27 1.27)) (justify left))
     )
-    (property "Value" "10k" (id 1) (at 38.1 30.4799 0)
-      (effects (font (size 1.27 1.27)) (justify left))
-    )
-    (property "Footprint" "Resistor_SMD:R_0402_1005Metric" (id 2) (at 35.56 29.21 0)
+    (property "Value" "" (id 1) (at 38.1 30.4799 0)
+      (effects (font (size 1.27 1.27)) (justify left))
+    )
+    (property "Footprint" "" (id 2) (at 35.56 29.21 0)
       (effects (font (size 1.27 1.27)) hide)
     )
@@
       (effects (font (size 1.27 1.27)) hide)
     )
-    (property "LCSC" "C25744" (id 4) (at 35.56 29.21 0)
+    (property "LCSC" "C11702" (id 4) (at 35.56 29.21 0)
       (effects (font (size 1.27 1.27)) hide)
     )
@@
     )
     (path "/40715f59-6f0a-47d8-b499-b0fd39ab216d"
-      (reference "R2") (unit 1) (value "10k") (footprint "Resistor_SMD:R_0402_1005Metric")
+      (reference "R2") (unit 1) (value "1k") (footprint "Resistor_SMD:R_0402_1005Metric")
     )
     (path "/7bb37abf-e644-464a-9660-0f67661d674a"
